Commit message: Functioning package

File: ws_description/urdf/panda_arm_hand.urdf.xacro (robot description, xacro)
@@ -74,10 +74,23 @@
     <parent link="panda_link8"/>
     <child link="camera_robot_"/>
-    <origin xyz="0 0.0 0.0" rpy="0 0 ${-pi/4}"/>
+    <origin xyz="0 0.0 0.0" rpy="0 0 ${-pi/4}"/> <!-- rpy= "0 0 ${-pi/4}" -->
   </joint>
   <xacro:include filename="$(find ws_description)/urdf/_d435.urdf.xacro"/>
   <xacro:sensor_d435 parent="camera_robot_" prefix="camera_robot_">
-    <origin xyz="0.063 0 0" rpy="0 0 0"/>
+    <origin xyz="0.063 0 0.0125" rpy="0 ${-pi/2} ${pi}"/>
   </xacro:sensor_d435>
+  <link name="panda_arm_ee_link">
+    <visual>
+      <geometry>
+        <box size="0 0 0"/>
+      </geometry>
+      <origin xyz = "0 0 0" rpy = "0 0 0"/>
+    </visual>
+  </link>
+  <joint name="panda_arm_ee" type="fixed">
+    <parent link="panda_link8"/>
+    <child link="panda_arm_ee_link"/>
+    <origin xyz="0 0.0 0.1034" rpy="0 0 ${-pi/4}"/> <!-- rpy= "0 0 ${-pi/4}" -->
+  </joint>
   <!-- WORK TABLE -->
   <link name="table">

Commit message: changed moveit robotstate message

File: ws_description/urdf/panda_arm_hand.urdf.xacro (robot description, xacro)
@@ -200,5 +200,5 @@
       <visual>
         <geometry>
-          <box size="0.06 0.06 0.06"/>
+          <box size="0.16 0.16 0.16"/>
         </geometry>
         <origin rpy="0 0 0" xyz="0 0 0.0"/>
@@ -207,5 +207,5 @@
       <collision>
         <geometry>
-          <box size="0.06 0.06 0.06"/>
+          <box size="0.16 0.16 0.16"/>
         </geometry>
         <origin rpy="0 0 0" xyz="0 0 0.0"/>
@@ -241,5 +241,5 @@
       <visual>
         <geometry>
-          <box size="0.03 0.09 0.025"/>
+          <box size="0.2 0.2 0.2"/>
         </geometry>
         <origin rpy="0 0 0" xyz="0 0 0"/>
@@ -248,5 +248,5 @@
       <collision>
         <geometry>
-          <box size="0.03 0.09 0.025"/>
+          <box size="0.2 0.2 0.2"/>
         </geometry>
         <origin rpy="0 0 0" xyz="0 0 0"/>
